File: hardware/LEC000043.kicad_sch (KiCad schematic)
At the start: 54 parts, among them J1 FORCE_ACTIVATION, J2 TRACKS_OUT, J3 TRACKS_IN, J5 CONTACT_1, J6 CONTACT_2, K1 HK19F-5V, Q1 S8050, U1 NE555, U2 CYPC817, U3 XL1509-ADJE1

Commit message: Add prod files
Parts:
- C4, C9, LOGO1: now left out of the parts list
- J5, J6: JLCPCB_CORRECTION 0;0;180 -> 5.080;0;180
- RV1: JLCPCB_CORRECTION (none) -> 0;-1.27;0
Changed lines of the file:
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@@
       (effects (font (size 1.27 1.27)) hide)
     )
-    (property "JLCPCB_CORRECTION" "0;0;180" (id 9) (at 265.43 69.85 0)
+    (property "JLCPCB_CORRECTION" "5.080;0;180" (id 9) (at 265.43 69.85 0)
       (effects (font (size 1.27 1.27)) hide)
     )
@@
       (effects (font (size 1.27 1.27)) hide)
     )
-    (property "JLCPCB_CORRECTION" "0;0;180" (id 9) (at 265.43 81.28 0)
+    (property "JLCPCB_CORRECTION" "5.080;0;180" (id 9) (at 265.43 81.28 0)
       (effects (font (size 1.27 1.27)) hide)
     )
@@
   )
   (symbol (lib_id "Device:C_Small") (at 101.6 165.1 0) (unit 1)
-    (in_bom yes) (on_board yes)
+    (in_bom no) (on_board yes)
     (property "Reference" "C4" (id 0) (at 103.9368 163.9316 0)
       (effects (font (size 1.27 1.27)) (justify left))
@@
   )
   (symbol (lib_id "0_logos:logo_lectix_25mm") (at 222.25 173.99 0) (unit 1)
-    (in_bom yes) (on_board yes)
+    (in_bom no) (on_board yes)
     (property "Reference" "LOGO1" (id 0) (at 222.25 175.768 0)
       (effects (font (size 1.524 1.524)) hide)
@@
       (effects (font (size 1.27 1.27)) hide)
     )
+    (property "JLCPCB_CORRECTION" "0;-1.27;0" (id 7) (at 134.62 72.39 0)
+      (effects (font (size 1.27 1.27)) hide)
+    )
     (pin "1")
     (pin "2")
@@
   )
   (symbol (lib_id "Device:C") (at 107.95 107.95 0) (unit 1)
-    (in_bom yes) (on_board yes)
+    (in_bom no) (on_board yes)
     (property "Reference" "C9" (id 0) (at 110.871 106.7816 0)
       (effects (font (size 1.27 1.27)) (justify left))
